Commit message: Fix xacro symbol conflict preventing robot spawn
Remove duplicate 'pi' property definitions from gripper xacro files
that were causing "redefining global symbol" errors during xacro
processing. The 'pi' constant was defined but never used in these files.

This fixes the robot not spawning in Gazebo due to failed URDF generation.

File: husky_ur3_gazebo/urdf/rh_p12_rn.xacro (robot description, xacro)
@@ -1,6 +1,4 @@
 <?xml version="1.0"?>
 <robot name="rh_p12_rn" xmlns:xacro="http://www.ros.org/wiki/xacro">
-  <!-- some parameters -->
-  <xacro:property name="pi" value="3.141592654" />
   <!-- Import all Gazebo-customization elements, including Gazebo colors -->
   <xacro:include filename="$(find husky_ur3_gazebo)/urdf/rh_p12_rn.gazebo" />

File: husky_ur3_gazebo/urdf/rh_p12_rn_gripper.xacro (robot description, xacro)
@@ -2,6 +2,4 @@
 <robot name="rh_p12_rn" xmlns:xacro="http://www.ros.org/wiki/xacro">
 <!-- 210927 YSW: Added hardware interface and modified type of joints -->
-  <!-- some parameters -->
-  <xacro:property name="pi" value="3.141592654" />
   <!-- Import all Gazebo-customization elements, including Gazebo colors -->
   <xacro:include filename="$(find husky_ur3_gazebo)/urdf/rh_p12_rn.gazebo" />
