Commit message: Migrate husky_ur3_gazebo package from ROS1 to ROS2
This commit completes the migration of the package to ROS2 Humble:

Build System:
- Updated package.xml from format 2 (catkin) to format 3 (ament_cmake)
- Updated CMakeLists.txt to use ament_cmake instead of catkin
- Changed dependencies from ROS1 to ROS2 equivalents

URDF/Gazebo Plugins:
- Replaced libgazebo_ros_control.so with libgazebo_ros2_control.so
- Updated IMU plugin from libhector_gazebo_ros_imu.so to libgazebo_ros_imu_sensor.so
- Updated GPS plugin from libhector_gazebo_ros_gps.so to libgazebo_ros_gps_sensor.so
- Updated laser plugin from libgazebo_ros_laser.so to libgazebo_ros_ray_sensor.so
- Updated camera plugins from libgazebo_ros_openni_kinect.so to libgazebo_ros_camera.so

Mesh Files:
- Fixed RealSense D435 mesh paths from package://realsense2_description to package://husky_ur3_gazebo

Controllers:
- Updated control.yaml to ROS2 ros2_control format
- Updated controller types to ROS2 equivalents
- Added ros__parameters namespacing for ROS2 compatibility

Launch Files:
- Created test_urdf.launch.py for ROS2 launch system
- Includes Gazebo server/client, robot state publisher, and entity spawning

This migration addresses all the issues causing the original failure.

File: husky_ur3_gazebo/urdf/accessories/d435_camera_g.urdf.xacro (robot description, xacro)
@@ -54,5 +54,5 @@
         <geometry>
           <!-- <box size="${d435_cam_width} ${d435_cam_height} ${d435_cam_depth}"/> -->
-	        <mesh filename="package://realsense2_description/meshes/d435.dae" />
+	        <mesh filename="package://husky_ur3_gazebo/meshes/accessories/d435.dae" />
         </geometry>
         <material name ="white">
@@ -138,5 +138,6 @@
             <always_on>1</always_on>
             <visualize>true</visualize>
-            <camera>
+            <update_rate>20.0</update_rate>
+            <camera name="g_camera">
                 <horizontal_fov>${60*M_PI/180.0}</horizontal_fov>
                 <image>
@@ -145,32 +146,27 @@
                     <format>R8G8B8</format>
                 </image>
-                <depth_camera>
-                </depth_camera>
                 <clip>
                     <near>0.11</near>
                     <far>10</far>
                 </clip>
+                <noise>
+                    <type>gaussian</type>
+                    <mean>0.0</mean>
+                    <stddev>0.007</stddev>
+                </noise>
             </camera>
-            <plugin name="g_camera_controller" filename="libgazebo_ros_openni_kinect.so">
-                <alwaysOn>true</alwaysOn>
-                    <updateRate>20.0</updateRate>
-                    <cameraName>g_d435</cameraName>
-                    <frameName>g_camera_depth_optical_frame</frameName>
-                <imageTopicName>rgb/g_image_raw</imageTopicName>
-                <depthImageTopicName>depth/g_image_raw</depthImageTopicName>
-                <pointCloudTopicName>depth/g_points</pointCloudTopicName>
-                <cameraInfoTopicName>rgb/camera_info</cameraInfoTopicName>
-                <depthImageCameraInfoTopicName>depth/camera_info</depthImageCameraInfoTopicName>
-                <pointCloudCutoff>0.4</pointCloudCutoff>
-                    <hackBaseline>0.07</hackBaseline>
-                    <distortionK1>0.0</distortionK1>
-                    <distortionK2>0.0</distortionK2>
-                    <distortionK3>0.0</distortionK3>
-                    <distortionT1>0.0</distortionT1>
-                    <distortionT2>0.0</distortionT2>
-                <CxPrime>0.0</CxPrime>
-                <Cx>0.0</Cx>
-                <Cy>0.0</Cy>
-                <focalLength>0.0</focalLength>
+            <plugin name="g_camera_controller" filename="libgazebo_ros_camera.so">
+                <ros>
+                    <namespace>/g_d435</namespace>
+                    <remapping>~/image_raw:=rgb/image_raw</remapping>
+                    <remapping>~/depth/image_raw:=depth/image_raw</remapping>
+                    <remapping>~/depth/points:=depth/points</remapping>
+                    <remapping>~/camera_info:=rgb/camera_info</remapping>
+                    <remapping>~/depth/camera_info:=depth/camera_info</remapping>
+                </ros>
+                <camera_name>g_d435</camera_name>
+                <frame_name>g_camera_depth_optical_frame</frame_name>
+                <hack_baseline>0.07</hack_baseline>
+                <min_depth>0.4</min_depth>
             </plugin>
         </sensor>

File: husky_ur3_gazebo/urdf/accessories/d435_camera_h.urdf.xacro (robot description, xacro)
@@ -54,5 +54,5 @@
         <geometry>
           <!-- <box size="${d435_cam_width} ${d435_cam_height} ${d435_cam_depth}"/> -->
-	        <mesh filename="package://realsense2_description/meshes/d435.dae" />
+	        <mesh filename="package://husky_ur3_gazebo/meshes/accessories/d435.dae" />
         </geometry>
         <material name ="white">
@@ -138,5 +138,6 @@
             <always_on>1</always_on>
             <visualize>true</visualize>
-            <camera>
+            <update_rate>20.0</update_rate>
+            <camera name="h_camera">
                 <horizontal_fov>${60*M_PI/180.0}</horizontal_fov>
                 <image>
@@ -145,32 +146,27 @@
                     <format>R8G8B8</format>
                 </image>
-                <depth_camera>
-                </depth_camera>
                 <clip>
                     <near>0.11</near>
                     <far>10</far>
                 </clip>
+                <noise>
+                    <type>gaussian</type>
+                    <mean>0.0</mean>
+                    <stddev>0.007</stddev>
+                </noise>
             </camera>
-            <plugin name="h_camera_controller" filename="libgazebo_ros_openni_kinect.so">
-                <alwaysOn>true</alwaysOn>
-                    <updateRate>20.0</updateRate>
-                    <cameraName>h_d435</cameraName>
-                    <frameName>h_camera_depth_optical_frame</frameName>
-                <imageTopicName>rgb/h_image_raw</imageTopicName>
-                <depthImageTopicName>depth/h_image_raw</depthImageTopicName>
-                <pointCloudTopicName>depth/h_points</pointCloudTopicName>
-                <cameraInfoTopicName>rgb/camera_info</cameraInfoTopicName>
-                <depthImageCameraInfoTopicName>depth/camera_info</depthImageCameraInfoTopicName>
-                <pointCloudCutoff>0.4</pointCloudCutoff>
-                    <hackBaseline>0.07</hackBaseline>
-                    <distortionK1>0.0</distortionK1>
-                    <distortionK2>0.0</distortionK2>
-                    <distortionK3>0.0</distortionK3>
-                    <distortionT1>0.0</distortionT1>
-                    <distortionT2>0.0</distortionT2>
-                <CxPrime>0.0</CxPrime>
-                <Cx>0.0</Cx>
-                <Cy>0.0</Cy>
-                <focalLength>0.0</focalLength>
+            <plugin name="h_camera_controller" filename="libgazebo_ros_camera.so">
+                <ros>
+                    <namespace>/h_d435</namespace>
+                    <remapping>~/image_raw:=rgb/image_raw</remapping>
+                    <remapping>~/depth/image_raw:=depth/image_raw</remapping>
+                    <remapping>~/depth/points:=depth/points</remapping>
+                    <remapping>~/camera_info:=rgb/camera_info</remapping>
+                    <remapping>~/depth/camera_info:=depth/camera_info</remapping>
+                </ros>
+                <camera_name>h_d435</camera_name>
+                <frame_name>h_camera_depth_optical_frame</frame_name>
+                <hack_baseline>0.07</hack_baseline>
+                <min_depth>0.4</min_depth>
             </plugin>
         </sensor>

File: husky_ur3_gazebo/urdf/accessories/sick_tim571.urdf.xacro (robot description, xacro)
@@ -61,7 +61,11 @@
 					</noise>
 				</ray>
-				<plugin name="${prefix}_controller" filename="libgazebo_ros_laser.so">
-					<topicName>/scan</topicName>
-					<frameName>/${prefix}_link</frameName>
+				<plugin name="${prefix}_controller" filename="libgazebo_ros_ray_sensor.so">
+					<ros>
+						<namespace>/</namespace>
+						<remapping>~/out:=scan</remapping>
+					</ros>
+					<output_type>sensor_msgs/LaserScan</output_type>
+					<frame_name>${prefix}_link</frame_name>
 				</plugin>
 			</sensor>

File: husky_ur3_gazebo/urdf/husky_ur3_gripper.urdf.xacro (robot description, xacro)
@@ -184,36 +184,74 @@
   </gazebo>
   <gazebo>
-    <plugin name="gazebo_ros_control" filename="libgazebo_ros_control.so">
-      <robotNamespace>$(arg robot_namespace)</robotNamespace>
+    <plugin name="gazebo_ros2_control" filename="libgazebo_ros2_control.so">
+      <parameters>$(find husky_ur3_gazebo)/config/control.yaml</parameters>
     </plugin>
   </gazebo>
-  <gazebo>
-    <plugin name="imu_controller" filename="libhector_gazebo_ros_imu.so">
-      <robotNamespace>$(arg robot_namespace)</robotNamespace>
-      <updateRate>50.0</updateRate>
-      <bodyName>base_link</bodyName>
-      <topicName>imu/data</topicName>
-      <accelDrift>0.005 0.005 0.005</accelDrift>
-      <accelGaussianNoise>0.005 0.005 0.005</accelGaussianNoise>
-      <rateDrift>0.005 0.005 0.005 </rateDrift>
-      <rateGaussianNoise>0.005 0.005 0.005 </rateGaussianNoise>
-      <headingDrift>0.005</headingDrift>
-      <headingGaussianNoise>0.005</headingGaussianNoise>
-    </plugin>
-  </gazebo>
-  <gazebo>
-    <plugin name="gps_controller" filename="libhector_gazebo_ros_gps.so">
-      <robotNamespace>$(arg robot_namespace)</robotNamespace>
-      <updateRate>40</updateRate>
-      <bodyName>base_link</bodyName>
-      <frameId>base_link</frameId>
-      <topicName>navsat/fix</topicName>
-      <velocityTopicName>navsat/vel</velocityTopicName>
-      <referenceLatitude>49.9</referenceLatitude>
-      <referenceLongitude>8.9</referenceLongitude>
-      <referenceHeading>0</referenceHeading>
-      <referenceAltitude>0</referenceAltitude>
-      <drift>0.0001 0.0001 0.0001</drift>
-    </plugin>
+  <gazebo reference="imu_link">
+    <sensor name="imu_sensor" type="imu">
+      <always_on>true</always_on>
+      <update_rate>50</update_rate>
+      <imu>
+        <angular_velocity>
+          <x>
+            <noise type="gaussian">
+              <mean>0.0</mean>
+              <stddev>0.005</stddev>
+            </noise>
+          </x>
+          <y>
+            <noise type="gaussian">
+              <mean>0.0</mean>
+              <stddev>0.005</stddev>
+            </noise>
+          </y>
+          <z>
+            <noise type="gaussian">
+              <mean>0.0</mean>
+              <stddev>0.005</stddev>
+            </noise>
+          </z>
+        </angular_velocity>
+        <linear_acceleration>
+          <x>
+            <noise type="gaussian">
+              <mean>0.0</mean>
+              <stddev>0.005</stddev>
+            </noise>
+          </x>
+          <y>
+            <noise type="gaussian">
+              <mean>0.0</mean>
+              <stddev>0.005</stddev>
+            </noise>
+          </y>
+          <z>
+            <noise type="gaussian">
+              <mean>0.0</mean>
+              <stddev>0.005</stddev>
+            </noise>
+          </z>
+        </linear_acceleration>
+      </imu>
+      <plugin name="imu_plugin" filename="libgazebo_ros_imu_sensor.so">
+        <ros>
+          <namespace>/</namespace>
+          <remapping>~/out:=imu/data</remapping>
+        </ros>
+        <initial_orientation_as_reference>false</initial_orientation_as_reference>
+      </plugin>
+    </sensor>
+  </gazebo>
+  <gazebo reference="base_link">
+    <sensor name="gps_sensor" type="gps">
+      <always_on>true</always_on>
+      <update_rate>40</update_rate>
+      <plugin name="gps_plugin" filename="libgazebo_ros_gps_sensor.so">
+        <ros>
+          <namespace>/</namespace>
+          <remapping>~/out:=navsat/fix</remapping>
+        </ros>
+      </plugin>
+    </sensor>
   </gazebo>
   <!-- Optional custom includes. -->
